File: KiCad/AMS-Master.kicad_sch (KiCad schematic)
At the start: 33 parts, among them J7 JTAG, J8 DEBUG, SW1 MCU Reset, U7 IP4220CZ6, U8 FS32K148UJT0VLQT, Y1 8 MHz

Commit message: Port to Kicad 7, small changes in auto-reset feature
Connections:
- net AUTO_RESET_EN: now reaches U8.112 (PTD28)
- no-connect marks 68 -> 67
