File: KiCad/spr23e-bmu.kicad_pcb (KiCad board)
At the start: 4 copper layers, 157 x 100 mm, 433 parts, among them J1 LV_IO, J2 LV ACCU, J3 SENSOR, J4 TS, J5 ISO, J6 UART, J7 JTAG, J8 DEBUG, J9 Molex 104031-0811, Q1 SQ2308CES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

Commit message: Update KiCad project to newest version
Parts:
- R49, R50, R51, R52, R54, R55, R56, R57: value 680k -> 750k 0.1%
- R53, R58: value 9k1 -> 10k 0.1%
